File: board/board.kicad_sch (KiCad schematic)
At the start: 1 part

Commit message: initial
Parts:
- added J1: 009_1000BASE-T, on_edge:on_edge_2x05_device, symbol put_on_edge:009_1000BASE-T
- added R1: 0R, Resistor_SMD:R_0603_1608Metric, symbol Device:R_Small
Connections:
- new net Earth: J1.1 (GND), J1.6 (GND), R1.2
- new net rj45/SCHIELD: R1.1
- new net rj45/TD1+: J1.2 (TD1+)
- new net rj45/TD1-: J1.3 (TD1-)
- new net rj45/TD2+: J1.4 (TD2+)
- new net rj45/TD2-: J1.5 (TD2-)
- new net rj45/TD3+: J1.7 (TD3+)
- new net rj45/TD3-: J1.8 (TD3-)
- new net rj45/TD4+: J1.9 (TD4+)
- new net rj45/TD4-: J1.10 (TD4-)
Other:
- removed sheet implementation
- added sheet rj45 (rj45.kicad_sch)
- note removed: "Input connectors go here"
- note removed: "Output connectors go here"
Changed lines of the file:
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@@
 (kicad_sch (version 20211123) (generator eeschema)
   (paper "A4")
-  (text "Output connectors go here" (at 224.79 88.9 0)
-    (effects (font (size 1.27 1.27)) (justify left bottom))
+  (junction (at 85.09 104.775) (diameter 0) (color 0 0 0 0)
   )
-  (text "Input connectors go here" (at 49.53 88.9 0)
-    (effects (font (size 1.27 1.27)) (justify left bottom))
+  (junction (at 85.09 107.95) (diameter 0) (color 0 0 0 0)
+  )
+  (wire (pts (xy 96.52 83.82) (xy 111.76 83.82))
+    (stroke (width 0) (type default) (color 0 0 0 0))
+  )
+  (wire (pts (xy 85.09 104.775) (xy 86.36 104.775))
+    (stroke (width 0) (type default) (color 0 0 0 0))
+  )
+  (wire (pts (xy 96.52 93.98) (xy 111.76 93.98))
+    (stroke (width 0) (type default) (color 0 0 0 0))
+  )
+  (wire (pts (xy 83.82 104.14) (xy 83.82 104.775))
+    (stroke (width 0) (type default) (color 0 0 0 0))
+  )
+  (wire (pts (xy 100.33 107.95) (xy 111.76 107.95))
+    (stroke (width 0) (type default) (color 0 0 0 0))
+  )
+  (wire (pts (xy 86.36 104.775) (xy 86.36 104.14))
+    (stroke (width 0) (type default) (color 0 0 0 0))
+  )
+  (wire (pts (xy 96.52 99.06) (xy 111.76 99.06))
+    (stroke (width 0) (type default) (color 0 0 0 0))
+  )
+  (wire (pts (xy 96.52 86.36) (xy 111.76 86.36))
+    (stroke (width 0) (type default) (color 0 0 0 0))
+  )
+  (wire (pts (xy 83.82 104.775) (xy 85.09 104.775))
+    (stroke (width 0) (type default) (color 0 0 0 0))
+  )
+  (wire (pts (xy 96.52 91.44) (xy 111.76 91.44))
+    (stroke (width 0) (type default) (color 0 0 0 0))
+  )
+  (wire (pts (xy 85.09 109.22) (xy 85.09 107.95))
+    (stroke (width 0) (type default) (color 0 0 0 0))
+  )
+  (wire (pts (xy 96.52 96.52) (xy 111.76 96.52))
+    (stroke (width 0) (type default) (color 0 0 0 0))
+  )
+  (wire (pts (xy 85.09 107.95) (xy 95.25 107.95))
+    (stroke (width 0) (type default) (color 0 0 0 0))
+  )
+  (wire (pts (xy 96.52 88.9) (xy 111.76 88.9))
+    (stroke (width 0) (type default) (color 0 0 0 0))
+  )
+  (wire (pts (xy 96.52 81.28) (xy 111.76 81.28))
+    (stroke (width 0) (type default) (color 0 0 0 0))
+  )
+  (wire (pts (xy 85.09 107.95) (xy 85.09 104.775))
+    (stroke (width 0) (type default) (color 0 0 0 0))
+  )
+  (symbol (lib_id "put_on_edge:009_1000BASE-T") (at 85.09 90.17 0) (mirror y) (unit 1)
+    (in_bom yes) (on_board yes) (fields_autoplaced)
+    (property "Reference" "J1" (id 0) (at 85.725 72.39 0))
+    (property "Value" "009_1000BASE-T" (id 1) (at 85.725 74.93 0))
+    (property "Footprint" "on_edge:on_edge_2x05_device" (id 2) (at 77.47 73.66 0)
+      (effects (font (size 1.27 1.27)) hide)
+    )
+    (property "Datasheet" "" (id 3) (at 77.47 73.66 0)
+      (effects (font (size 1.27 1.27)) hide)
+    )
+    (pin "1")
+    (pin "10")
+    (pin "2")
+    (pin "3")
+    (pin "4")
+    (pin "5")
+    (pin "6")
+    (pin "7")
+    (pin "8")
+    (pin "9")
+  )
+  (symbol (lib_id "Device:R_Small") (at 97.79 107.95 270) (unit 1)
+    (in_bom yes) (on_board yes)
+    (property "Reference" "R1" (id 0) (at 97.79 102.9716 90))
+    (property "Value" "0R" (id 1) (at 97.79 105.283 90))
+    (property "Footprint" "Resistor_SMD:R_0603_1608Metric" (id 2) (at 97.79 107.95 0)
+      (effects (font (size 1.27 1.27)) hide)
+    )
+    (property "Datasheet" "~" (id 3) (at 97.79 107.95 0)
+      (effects (font (size 1.27 1.27)) hide)
+    )
+    (pin "1")
+    (pin "2")
+  )
+  (symbol (lib_id "power:Earth") (at 85.09 109.22 0) (unit 1)
+    (in_bom yes) (on_board yes)
+    (property "Reference" "#PWR0101" (id 0) (at 85.09 115.57 0)
+      (effects (font (size 1.27 1.27)) hide)
+    )
+    (property "Value" "Earth" (id 1) (at 85.09 113.03 0)
+      (effects (font (size 1.27 1.27)) hide)
+    )
+    (property "Footprint" "" (id 2) (at 85.09 109.22 0)
+      (effects (font (size 1.27 1.27)) hide)
+    )
+    (property "Datasheet" "~" (id 3) (at 85.09 109.22 0)
+      (effects (font (size 1.27 1.27)) hide)
+    )
+    (pin "1")
   )
   (symbol (lib_id "Graphic:Logo_Open_Hardware_Small") (at 273.05 157.48 0) (unit 1)
@@
     )
   )
-  (sheet (at 114.3 72.39) (size 60.96 62.23) (fields_autoplaced)
+  (sheet (at 111.76 62.23) (size 45.72 53.34) (fields_autoplaced)
     (stroke (width 0.1524) (type solid) (color 0 0 0 0))
     (fill (color 0 0 0 0.0000))
-    (property "Sheet name" "implementation" (id 0) (at 114.3 71.6784 0)
+    (property "Sheet name" "rj45" (id 0) (at 111.76 61.5184 0)
       (effects (font (size 1.27 1.27)) (justify left bottom))
     )
-    (property "Sheet file" "implementation.kicad_sch" (id 1) (at 114.3 135.2046 0)
+    (property "Sheet file" "rj45.kicad_sch" (id 1) (at 111.76 116.1546 0)
       (effects (font (size 1.27 1.27)) (justify left top))
+    )
+    (pin "TD4-" input (at 111.76 99.06 180)
+      (effects (font (size 1.27 1.27)) (justify left))
+    )
+    (pin "TD4+" input (at 111.76 96.52 180)
+      (effects (font (size 1.27 1.27)) (justify left))
+    )
+    (pin "TD1+" input (at 111.76 81.28 180)
+      (effects (font (size 1.27 1.27)) (justify left))
+    )
+    (pin "TD2+" input (at 111.76 86.36 180)
+      (effects (font (size 1.27 1.27)) (justify left))
+    )
+    (pin "TD3-" input (at 111.76 93.98 180)
+      (effects (font (size 1.27 1.27)) (justify left))
+    )
+    (pin "SCHIELD" input (at 111.76 107.95 180)
+      (effects (font (size 1.27 1.27)) (justify left))
+    )
+    (pin "TD3+" input (at 111.76 91.44 180)
+      (effects (font (size 1.27 1.27)) (justify left))
+    )
+    (pin "TD2-" input (at 111.76 88.9 180)
+      (effects (font (size 1.27 1.27)) (justify left))
+    )
+    (pin "TD1-" input (at 111.76 83.82 180)
+      (effects (font (size 1.27 1.27)) (justify left))
     )
   )
   (sheet_instances
     (path "/" (page "1"))
-    (path "/767ce4c6-0e55-4543-92f0-34cb8237a544" (page "2"))
+    (path "/2366e56d-f0ca-498c-aaf9-0ba2aaf17538" (page "2"))
   )
   (symbol_instances
+    (path "/75462683-7040-4b5b-8fc2-30b8f3d83ab4"
+      (reference "#PWR0101") (unit 1) (value "Earth") (footprint "")
+    )
+    (path "/32a88e68-75fd-45a8-8ae7-e79098a66cab"
+      (reference "J1") (unit 1) (value "009_1000BASE-T") (footprint "on_edge:on_edge_2x05_device")
+    )
+    (path "/2366e56d-f0ca-498c-aaf9-0ba2aaf17538/8ace62d9-8060-4514-b211-5041041f8626"
+      (reference "J2") (unit 1) (value "615008145521") (footprint "b010:RJ45_Wuerth_615008145521_Horizontal")
+    )
     (path "/b72b6f4a-7489-40f2-bb90-d75ae01aa368"
       (reference "LOGO1") (unit 1) (value "Logo_Open_Hardware_Small") (footprint "Symbol:OSHW-Symbol_6.7x6mm_SilkScreen")
     )
+    (path "/45d557d0-55c0-4c2d-b60b-202523ab9de1"
+      (reference "R1") (unit 1) (value "0R") (footprint "Resistor_SMD:R_0603_1608Metric")
+    )
   )
